File: pcb_files/mouse/mouse_v2.sch (KiCad schematic (older format))
At the start: 56 parts, among them J4 I2C_Conn, M1 Motor_DC, M2 Motor_DC, Q0 Q_Photo_NPN, Q1 Q_Photo_NPN, Q2 Q_Photo_NPN, Q3 Q_Photo_NPN, T0 Q_NMOS_DGS, T1 Q_NMOS_DGS, T2 Q_NMOS_DGS, T3 Q_NMOS_DGS, U1 Teensy4.0, U2 SN754410NE (Half-Bridge), U3 LM1085-5.0, U4 Encoder_3081, U5 Encoder_3081

Commit message: Updated pins for Teensy, pre traces
Connections:
- net Buzzer: now also U1.4 (2_OUT2); no longer U1.13 (11_MOSI_CTX1)
- net Emitter_1: now also U1.28 (21_A7_RX5_BCLK1); no longer U1.27 (20_A6_TX5_LRCLK1)
- net Emitter_2: now also U1.21 (14_A0_TX3_SPDIF_OUT); no longer U1.22 (15_A1_RX3_SPDIF_IN)
- net Emitter_3: now also U1.25 (18_A4_SDA0); no longer U1.24 (17_A3_TX4_SDA1)
- net LED_1: now also U1.7 (5_IN2); no longer U1.20 (13_SCK_CRX1_LED)
- net LED_2: now also U1.5 (3_LRCLK2); no longer U1.25 (18_A4_SDA0)
- net LED_3: now also U1.6 (4_BCLK2); no longer U1.26 (19_A5_SCL0)
- net M1_backward: now also U1.11 (9_OUT1C); no longer U1.2 (0_RX1_CRX2_CS1)
- net M1_encoder_A: now also U1.24 (17_A3_TX4_SDA1); no longer U1.10 (8_TX2_IN1)
- net M1_encoder_B: now also U1.23 (16_A2_RX4_SCL1); no longer U1.11 (9_OUT1C)
- net M1_forward: now also U1.13 (11_MOSI_CTX1); no longer U1.3 (1_TX1_CTX2_MISO1)
- net M1_speed: now also U1.14 (12_MISO_MQSL); no longer U1.6 (4_BCLK2)
- net M2_backward: now also U1.10 (8_TX2_IN1); no longer U1.5 (3_LRCLK2)
- net M2_encoder_A: now also U1.3 (1_TX1_CTX2_MISO1); no longer U1.9 (7_RX2_OUT1A)
- net M2_encoder_B: now also U1.2 (0_RX1_CRX2_CS1); no longer U1.8 (6_OUT1D)
- net M2_forward: now also U1.9 (7_RX2_OUT1A); no longer U1.4 (2_OUT2)
- net M2_speed: now also U1.8 (6_OUT1D); no longer U1.7 (5_IN2)
- net PUSH_SW: now also U1.22 (15_A1_RX3_SPDIF_IN); no longer U1.14 (12_MISO_MQSL)
- net Reciever_1: now also U1.27 (20_A6_TX5_LRCLK1); no longer U1.28 (21_A7_RX5_BCLK1)
- net Reciever_2: now also U1.20 (13_SCK_CRX1_LED); no longer U1.21 (14_A0_TX3_SPDIF_OUT)
- net Reciever_3: now also U1.26 (19_A5_SCL0); no longer U1.23 (16_A2_RX4_SCL1)
Changed lines of the file:
@@
 Text Label 4400 10050 2    50   ~ 0
 GND
-Text Label 7600 1425 2    50   ~ 0
+Text Label 7600 2225 2    50   ~ 0
 M1_speed
-Text Label 7600 1525 2    50   ~ 0
+Text Label 7600 1625 2    50   ~ 0
 M2_speed
 Text Label 6100 8800 0    50   ~ 0
@@
 Text Label 9800 3525 0    50   ~ 0
 Reciever_0
-Text Label 7600 3625 2    50   ~ 0
+Text Label 7600 3525 2    50   ~ 0
 Reciever_1
-Text Label 7600 2925 2    50   ~ 0
+Text Label 7600 2825 2    50   ~ 0
 Reciever_2
-Text Label 7600 3125 2    50   ~ 0
+Text Label 7600 3425 2    50   ~ 0
 Reciever_3
 Text Label 9800 3625 0    50   ~ 0
 Emitter_0
-Text Label 7600 3525 2    50   ~ 0
+Text Label 7600 3625 2    50   ~ 0
 Emitter_1
-Text Label 7600 3025 2    50   ~ 0
+Text Label 7600 2925 2    50   ~ 0
 Emitter_2
-Text Label 7600 3225 2    50   ~ 0
+Text Label 7600 3325 2    50   ~ 0
 Emitter_3
-Text Label 7600 1125 2    50   ~ 0
+Text Label 7600 2125 2    50   ~ 0
 M1_forward
-Text Label 7600 1025 2    50   ~ 0
+Text Label 7600 1925 2    50   ~ 0
 M1_backward
-Text Label 7600 1225 2    50   ~ 0
+Text Label 7600 1725 2    50   ~ 0
 M2_forward
-Text Label 7600 1325 2    50   ~ 0
+Text Label 7600 1825 2    50   ~ 0
 M2_backward
 Text Label 8225 4650 3    50   ~ 0
@@
 Wire Wire Line
 	8275 4125 8450 4125
-Text Label 7600 1825 2    50   ~ 0
+Text Label 7600 3225 2    50   ~ 0
 M1_encoder_A
-Text Label 7600 1925 2    50   ~ 0
+Text Label 7600 3125 2    50   ~ 0
 M1_encoder_B
-Text Label 7600 1725 2    50   ~ 0
+Text Label 7600 1125 2    50   ~ 0
 M2_encoder_A
-Text Label 7600 1625 2    50   ~ 0
+Text Label 7600 1025 2    50   ~ 0
 M2_encoder_B
 NoConn ~ 9800 1025
 NoConn ~ 9800 1125
 NoConn ~ 9800 1225
-Text Label 7600 2225 2    50   ~ 0
+Text Label 7600 3025 2    50   ~ 0
 PUSH_SW
 Text Label 7600 925  2    50   ~ 0
@@
 Wire Wire Line
 	1175 6975 1350 6975
-Text Label 7600 3425 2    50   ~ 0
+Text Label 7600 1425 2    50   ~ 0
 LED_3
-Text Label 7600 3325 2    50   ~ 0
+Text Label 7600 1325 2    50   ~ 0
 LED_2
-Text Label 7600 2825 2    50   ~ 0
+Text Label 7600 1525 2    50   ~ 0
 LED_1
-Text Label 7600 2125 2    50   ~ 0
+Text Label 7600 1225 2    50   ~ 0
 Buzzer
 $EndSCHEMATC
