File: pcb_files/mouse/mouse_v2.sch (KiCad schematic (older format))
At the start: 56 parts, among them J4 I2C_Conn, M1 Motor_DC, M2 Motor_DC, Q0 Q_Photo_NPN, Q1 Q_Photo_NPN, Q2 Q_Photo_NPN, Q3 Q_Photo_NPN, T0 Q_NMOS_DGS, T1 Q_NMOS_DGS, T2 Q_NMOS_DGS, T3 Q_NMOS_DGS, U1 Teensy4.0, U2 SN754410NE (Half-Bridge), U3 LM1085-5.0, U4 Encoder_3081, U5 Encoder_3081

Commit message: Traces Complete
Parts:
- U1: footprint teensy:Teensy40 -> teensy:Teensy40(nopads)
Connections:
- net M1_backward: now also U1.10 (8_TX2_IN1); no longer U1.11 (9_OUT1C)
- net M2_backward: now also U1.11 (9_OUT1C); no longer U1.10 (8_TX2_IN1)
Changed lines of the file:
@@
 Text Label 7600 2125 2    50   ~ 0
 M1_forward
-Text Label 7600 1925 2    50   ~ 0
+Text Label 7600 1825 2    50   ~ 0
 M1_backward
 Text Label 7600 1725 2    50   ~ 0
 M2_forward
-Text Label 7600 1825 2    50   ~ 0
+Text Label 7600 1925 2    50   ~ 0
 M2_backward
 Text Label 8225 4650 3    50   ~ 0
@@
 F 0 "U1" H 8700 3890 50  0000 C CNN
 F 1 "Teensy4.0" H 8700 3799 50  0000 C CNN
-F 2 "teensy:Teensy40" H 8300 2475 50  0001 C CNN
+F 2 "teensy:Teensy40(nopads)" H 8300 2475 50  0001 C CNN
 F 3 "" H 8300 2475 50  0001 C CNN
 	1    8700 2275
