File: pcb_files/mouse/mouse_v2.sch (KiCad schematic (older format))
At the start: 67 parts, among them J1 Conn_01x06_Female, J2 Conn_01x02_Female, J4 I2C_Conn, M1 Motor_DC, M2 Motor_DC, Q0 Q_Photo_NPN, Q1 Q_Photo_NPN, Q2 Q_Photo_NPN, Q3 Q_Photo_NPN, T0 Q_NMOS_DGS, T1 Q_NMOS_DGS, T2 Q_NMOS_DGS, T3 Q_NMOS_DGS, T4 Q_NMOS_DGS, U1 Teensy4.0, U2 SN754410NE (Half-Bridge), U3 LM1085-5.0, U4 Encoder_3081, U5 Encoder_3081

Commit message: updates
Parts:
- gave numbers to parts that had none: 1
Changed lines of the file:
@@
 PUSH_SW2
 $Comp
-L Connector:Conn_01x02_Male J?
+L Connector:Conn_01x02_Male J3
 U 1 1 608D00EC
 P 7575 5625
-F 0 "J?" H 7683 5806 50  0000 C CNN
+F 0 "J3" H 7683 5806 50  0000 C CNN
 F 1 "Conn_01x02_Male" H 7683 5715 50  0000 C CNN
 F 2 "" H 7575 5625 50  0001 C CNN

Commit message: added hc05 key jumper
Parts:
- J3: footprint (none) -> Connector_PinHeader_2.54mm:PinHeader_1x02_P2.54mm_Vertical
Changed lines of the file:
@@
 F 0 "J3" H 7683 5806 50  0000 C CNN
 F 1 "Conn_01x02_Male" H 7683 5715 50  0000 C CNN
-F 2 "" H 7575 5625 50  0001 C CNN
+F 2 "Connector_PinHeader_2.54mm:PinHeader_1x02_P2.54mm_Vertical" H 7575 5625 50  0001 C CNN
 F 3 "~" H 7575 5625 50  0001 C CNN
 	1    7575 5625

Commit message: changed led to smaller footprint, generated gerbers
Parts:
- D4, D5, D6: footprint LED_SMD:LED_1206_3216Metric_Pad1.42x1.75mm_HandSolder -> LED_SMD:LED_0201_0603Metric_Pad0.64x0.40mm_HandSolder
Changed lines of the file:
@@
 F 0 "D4" H 2141 6516 50  0000 C CNN
 F 1 "LED" H 2141 6425 50  0000 C CNN
-F 2 "LED_SMD:LED_1206_3216Metric_Pad1.42x1.75mm_HandSolder" H 2150 6300 50  0001 C CNN
+F 2 "LED_SMD:LED_0201_0603Metric_Pad0.64x0.40mm_HandSolder" H 2150 6300 50  0001 C CNN
 F 3 "~" H 2150 6300 50  0001 C CNN
 	1    2150 6300
@@
 F 0 "D5" H 2141 7041 50  0000 C CNN
 F 1 "LED" H 2141 6950 50  0000 C CNN
-F 2 "LED_SMD:LED_1206_3216Metric_Pad1.42x1.75mm_HandSolder" H 2150 6825 50  0001 C CNN
+F 2 "LED_SMD:LED_0201_0603Metric_Pad0.64x0.40mm_HandSolder" H 2150 6825 50  0001 C CNN
 F 3 "~" H 2150 6825 50  0001 C CNN
 	1    2150 6825
@@
 F 0 "D6" H 2141 7566 50  0000 C CNN
 F 1 "LED" H 2141 7475 50  0000 C CNN
-F 2 "LED_SMD:LED_1206_3216Metric_Pad1.42x1.75mm_HandSolder" H 2150 7350 50  0001 C CNN
+F 2 "LED_SMD:LED_0201_0603Metric_Pad0.64x0.40mm_HandSolder" H 2150 7350 50  0001 C CNN
 F 3 "~" H 2150 7350 50  0001 C CNN
 	1    2150 7350
