File: pcb_files/mouse/_saved_mouse_v2.sch (KiCad schematic (older format))
At the start: 57 parts, among them J4 I2C_Conn, M1 Motor_DC, M2 Motor_DC, Q0 Q_Photo_NPN, Q1 Q_Photo_NPN, Q2 Q_Photo_NPN, Q3 Q_Photo_NPN, T0 Q_NMOS_DGS, T1 Q_NMOS_DGS, T2 Q_NMOS_DGS, T3 Q_NMOS_DGS, U1 Teensy4.0, U2 SN754410NE (Half-Bridge), U3 LM1085-5.0, U4 Encoder_3081, U5 Encoder_3081

Commit message: Final Schematic and PCB changes
Parts:
- C1, C3: footprint (none) -> Capacitor_THT:CP_Radial_D5.0mm_P2.50mm
Changed lines of the file:
@@
 Text Label 4200 8600 2    50   ~ 0
-GND
-Text Label 4200 9100 3    50   ~ 0
 GND
 $Comp
@@
 F 0 "C3" H 4010 5854 50  0000 R CNN
 F 1 "100uF" H 4010 5945 50  0000 R CNN
-F 2 "" H 4125 5900 50  0001 C CNN
+F 2 "Capacitor_THT:CP_Radial_D5.0mm_P2.50mm" H 4125 5900 50  0001 C CNN
 F 3 "~" H 4125 5900 50  0001 C CNN
 	1    4125 5900
@@
 F 0 "C1" H 3535 5854 50  0000 R CNN
 F 1 "100uF" H 3535 5945 50  0000 R CNN
-F 2 "" H 3650 5900 50  0001 C CNN
+F 2 "Capacitor_THT:CP_Radial_D5.0mm_P2.50mm" H 3650 5900 50  0001 C CNN
 F 3 "~" H 3650 5900 50  0001 C CNN
 	1    3650 5900
