File: pcb_files/mouse/mouse_v2.kicad_pcb (KiCad board)
At the start: 2 copper layers, 84.9 x 94.9 mm, 58 parts, among them J4 I2C_Conn, M1 Motor_DC, M2 Motor_DC, Q0 Q_Photo_NPN, Q1 Q_Photo_NPN, Q2 Q_Photo_NPN, Q3 Q_Photo_NPN, T0 Q_NMOS_DGS, T1 Q_NMOS_DGS, T2 Q_NMOS_DGS, T3 Q_NMOS_DGS, U1 Teensy4.0, U2 SN754410NE (Half-Bridge), U3 LM1085-5.0, U4 Encoder_3081, U5 Encoder_3081

Commit message: added slot for bluetooth module
Parts:
- added J1: Conn_01x06_Female, Connector_PinHeader_2.54mm:PinHeader_1x06_P2.54mm_Vertical, F.Cu at (121.7, 120.1)
- added J2: Conn_01x02_Female, Connector_PinHeader_2.54mm:PinHeader_1x02_P2.54mm_Vertical, F.Cu at (156.9, 121.2)
- U1: footprint teensy:Teensy40(nopads) -> teensy:Teensy40
- moved SK1 0.38 mm to (160.1, 60.6)
- moved SK2 0.08 mm to (160.1, 141.0)
Routing:
- net /HC05_RX: track 0.00 -> 31.8 mm
- net /HC05_TX: track 0.00 -> 29.5 mm
- net /GND: track 15.9 -> 32.2 mm, vias 30 -> 41
- net /SCL2: track 0.00 -> 12.3 mm
- net /SDA2: track 0.00 -> 8.06 mm
- net /3.3v: track 176.8 -> 183.0 mm, vias 0 -> 1
- net Net-(D2-Pad1): track 27.3 -> 31.7 mm
- net /PUSH_SW: track 83.6 -> 82.7 mm
- net Net-(R11-Pad1): track 11.1 -> 11.7 mm

Commit message: rerouted traces, placed vol meter,
Parts:
- added R22: R, Resistor_THT:R_Axial_DIN0207_L6.3mm_D2.5mm_P10.16mm_Horizontal, F.Cu at (164.9, 79.7)
- added R23: R, Resistor_THT:R_Axial_DIN0207_L6.3mm_D2.5mm_P10.16mm_Horizontal, F.Cu at (168.2, 67.4)
- added SK3: M3, MountingHole:MountingHole_2.2mm_M2, F.Cu at (69.6, 62.5)
- added SK4: M3, MountingHole:MountingHole_2.2mm_M2, F.Cu at (75.6, 62.5)
- added T4: Q_NMOS_DGS, misc:TN0104(TO-92)v2, F.Cu at (150.3, 60.0)
- D4, D5, D6: footprint LED_THT:LED_D5.0mm -> LED_SMD:LED_1206_3216Metric_Pad1.42x1.75mm_HandSolder
- MH1, MH2, SK1, SK2: footprint MountingHole:MountingHole_3.2mm_M3 -> MountingHole:MountingHole_2.2mm_M2
- R17: value R_PULL_UP -> 47k; moved to B.Cu
- R18: moved to B.Cu
- R19: footprint Resistor_THT:R_Axial_DIN0207_L6.3mm_D2.5mm_P10.16mm_Horizontal -> Resistor_SMD:R_1206_3216Metric_Pad1.30x1.75mm_HandSolder
- R20, R21: footprint Resistor_THT:R_Axial_DIN0207_L6.3mm_D2.5mm_P10.16mm_Horizontal -> Resistor_SMD:R_1206_3216Metric_Pad1.30x1.75mm_HandSolder; moved to B.Cu
- moved BZ1 27.1 mm to (139.7, 60.1)
- moved R18 23.3 mm to (146.4, 59.9), turned to 180 degrees
- moved R21 16.7 mm to (121.4, 64.2)
- moved R20 16.1 mm to (121.7, 57.8)
- moved R19 13.7 mm to (124.6, 68.0)
- moved R17 10.6 mm to (136.3, 62.9)
- moved D4 0.90 mm to (120.4, 69.7)
Connections:
- BZ1 pad 1: Net-(BZ1-Pad1) -> /5v
- BZ1 pad 2: /GND -> Net-(BZ1-Pad2)
- J1 pad 5: /VCC -> /5v
- R17 pad 1: /PUSH_SW -> Net-(R17-Pad1)
- R17 pad 2: /3.3v -> /Buzzer
- R18 pad 1: /Buzzer -> Net-(BZ1-Pad2)
- R18 pad 2: Net-(BZ1-Pad1) -> Net-(R18-Pad2)
- U1 pad 41: Net-(U1-Pad41) -> /V_METER
Routing:
- net /V_METER: track 0.00 -> 67.5 mm, vias 0 -> 2
- net /3.3v: track 183.0 -> 127.6 mm
- net Net-(D6-Pad2): track 23.7 -> 0.00 mm
- net Net-(D4-Pad2): track 18.6 -> 0.00 mm
- net /LED_2: track 66.0 -> 48.2 mm
- net Net-(D5-Pad2): track 17.6 -> 0.00 mm
- net Net-(R17-Pad1): track 0.00 -> 16.3 mm
- net /LED_3: track 62.6 -> 46.6 mm
- net /M1_encoder_B: track 52.7 -> 68.5 mm
- net Net-(R18-Pad2): track 0.00 -> 15.1 mm
- net /Buzzer: track 47.2 -> 61.6 mm, vias 0 -> 1
- net Net-(BZ1-Pad1): track 13.9 -> 0.00 mm
- net /M1_encoder_A: track 52.8 -> 64.9 mm
- net /LED_1: track 59.5 -> 49.7 mm
- net Net-(BZ1-Pad2): track 0.00 -> 7.85 mm
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
Commit message: re-layout power section
Parts:
- C10: moved to F.Cu
- C2: moved to B.Cu
- moved C2 51.6 mm to (136.7, 65.5)
- moved C3 29.0 mm to (171.8, 68.8), turned to 180 degrees
- moved BT1 27.8 mm to (170.8, 73.7), turned to 90 degrees
- moved C1 18.2 mm to (171.8, 62.8), turned to 180 degrees
- moved J4 15.9 mm to (181.3, 74.5)
- moved S1 13.7 mm to (198.1, 58.4), turned to 270 degrees
- moved C10 12.4 mm to (193.1, 60.0), turned to 270 degrees
- moved U3 7.16 mm to (182.7, 62.8), turned to 0 degrees
- moved C9 7.04 mm to (176.7, 68.7), turned to 0 degrees
- moved R23 3.36 mm to (164.9, 67.2)
- moved BZ1 0.84 mm to (140.1, 59.4)
Routing:
- net /5v: track 445.2 -> 471.9 mm
- net /vBatt: track 69.5 -> 52.6 mm, vias 2 -> 1
- net /VUSB: track 83.9 -> 74.9 mm, vias 0 -> 1
- net /GND: track 32.2 -> 28.6 mm, vias 36 -> 33
- net Net-(C10-Pad1): track 26.5 -> 23.0 mm, vias 7 -> 9
- net /V_METER: track 67.5 -> 65.6 mm
- removed copper zone on B.Cu, net Net-(C10-Pad1)

Commit message: reworked power layout, added second button and key jumper to schem
Parts:
- R19: moved to B.Cu
- moved R19 3.25 mm to (121.9, 69.8)
- moved SK1 2.83 mm to (160.1, 57.8)
Routing:
- net /LED_2: track 48.2 -> 53.9 mm, vias 0 -> 1
- net /LED_3: track 46.6 -> 50.9 mm, vias 0 -> 1
- net /OUT3: track 23.0 -> 24.8 mm, vias 0 -> 1
- net /vBatt: track 52.6 -> 54.1 mm, vias 1 -> 0
- net /LED_1: track 49.7 -> 48.9 mm, vias 0 -> 1
- net /OUT4: vias 0 -> 1
- net /GND: vias 33 -> 29

Commit message: updates
Parts:
- added S3: GPTS203211B, Button_Switch_THT:SW_PUSH_6mm, F.Cu at (126.9, 65.0)
- R2, R4, R6, R8: moved to B.Cu
- moved D2 11.1 mm to (121.7, 121.0)
- moved D3 10.2 mm to (157.1, 142.4)
- moved D1 10.0 mm to (161.9, 144.5)
- moved Q2 5.07 mm to (130.2, 128.1)
- moved Q0 5.01 mm to (187.4, 128.3)
- moved D0 5.00 mm to (192.4, 128.3)
- moved D4 3.06 mm to (121.4, 66.8)
- moved R20 2.73 mm to (122.9, 60.2)
- moved D6 2.38 mm to (121.4, 62.2)
- moved J1 2.19 mm to (121.5, 117.9)
- moved C2 2.00 mm to (137.8, 67.2), turned to 270 degrees
- moved R21 1.61 mm to (122.9, 64.5)
- moved D5 1.44 mm to (121.4, 57.9)
- moved R19 1.27 mm to (122.9, 69.1)
- moved SK1 1.23 mm to (160.1, 59.0)
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Connections:
- net Net-(J1-Pad6) renamed /HC05_KEY
- U1 pad 12: Net-(U1-Pad12) -> /PUSH_SW2
- U1 pad 20: /Emitter_2 -> /PUSH_SW
- U1 pad 22: /PUSH_SW -> /Emitter_2
Routing:
- net /PUSH_SW2: track 0.00 -> 62.0 mm, vias 0 -> 1
- net /LED_2: track 53.9 -> 91.9 mm, vias 1 -> 2
- net /LED_1: track 48.9 -> 86.4 mm, vias 1 -> 2
- net /LED_3: track 50.9 -> 87.8 mm, vias 1 -> 2
- net /Emitter_2: track 28.4 -> 49.8 mm, vias 0 -> 1
- net /Buzzer: track 61.6 -> 78.6 mm
- net /5v: track 471.9 -> 483.9 mm
- net Net-(R11-Pad1): track 11.7 -> 4.97 mm
- net Net-(D6-Pad2): track 0.00 -> 2.93 mm, vias 0 -> 1
- net Net-(D5-Pad2): track 0.00 -> 2.93 mm, vias 0 -> 1
- net Net-(D4-Pad2): track 0.00 -> 2.93 mm, vias 0 -> 1
- net Net-(R7-Pad2): track 6.62 -> 4.83 mm
- net Net-(R17-Pad1): track 16.3 -> 15.4 mm
- net Net-(BZ1-Pad2): track 7.85 -> 7.18 mm
- net /GND: track 28.6 -> 28.5 mm, vias 29 -> 52
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
Commit message: reposition emitters
Parts:
- moved D0 7.95 mm to (195.9, 121.2)
- moved Q3 6.39 mm to (149.3, 139.7)
- moved Q1 6.37 mm to (169.7, 142.0)
- moved Q0 3.29 mm to (190.4, 127.1)
- moved Q2 3.28 mm to (127.2, 126.9)
- moved D3 0.08 mm to (157.1, 142.3)
Routing:
- net /GND: vias 52 -> 50
- net /5v: vias 1 -> 2

Commit message: fixed emiter/reciver traces
Parts:
- moved R2 0.76 mm to (164.6, 134.6)
- moved R4 0.74 mm to (155.5, 134.6)
Routing:
- net /3.3v: track 127.6 -> 74.0 mm
- net Net-(D0-Pad1): track 32.4 -> 16.9 mm
- net Net-(D2-Pad1): track 31.7 -> 17.3 mm
- net /5v: track 483.9 -> 496.6 mm
- net Net-(R11-Pad1): track 4.97 -> 11.8 mm
- net /Reciever_1: track 30.1 -> 25.2 mm
- net Net-(D3-Pad1): track 10.2 -> 5.71 mm
- net /Reciever_3: track 28.3 -> 25.0 mm
- net /HC05_TX: track 29.2 -> 32.4 mm
- net /HC05_RX: track 31.8 -> 34.0 mm
- net /Reciever_2: track 36.0 -> 34.0 mm
- net Net-(D1-Pad1): track 6.01 -> 7.59 mm
- net Net-(R7-Pad2): track 4.83 -> 5.80 mm
- net /Reciever_0: track 37.6 -> 38.3 mm
- net /HC05_KEY: vias 2 -> 0
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
Commit message: updates
Parts:
- moved J2 11.2 mm to (168.1, 121.2)
Routing:
- net /SCL2: track 12.3 -> 24.4 mm
- net /SDA2: track 8.06 -> 19.4 mm
Changed lines of the file:
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@@
     (thickness 1.6)
     (drawings 59)
-    (tracks 635)
+    (tracks 633)
     (zones 0)
     (modules 66)
@@
   )
   (module Connector_PinHeader_2.54mm:PinHeader_1x02_P2.54mm_Vertical (layer F.Cu)
-    (at 156.9212 121.2088 180)
+    (at 168.0972 121.158 180)
     (descr "Through hole straight pin header, 1x02, 2.54mm pitch, single row")
     (tags "Through hole pin header THT 1x02 2.54mm single row")
@@
   (segment (start 147.5844 120) (end 146.304 118.7196) (width 0.25) (layer F.Cu) (net 56))
   (segment (start 148.844 120) (end 147.5844 120) (width 0.25) (layer F.Cu) (net 56))
-  (segment (start 151.384 125.08) (end 152.8976 125.08) (width 0.25) (layer F.Cu) (net 57))
-  (segment (start 152.8976 125.08) (end 154.4828 123.4948) (width 0.25) (layer F.Cu) (net 57))
-  (segment (start 154.4828 123.4948) (end 154.4828 121.92) (width 0.25) (layer F.Cu) (net 57))
-  (segment (start 155.194 121.2088) (end 156.9212 121.2088) (width 0.25) (layer F.Cu) (net 57))
-  (segment (start 154.4828 121.92) (end 155.194 121.2088) (width 0.25) (layer F.Cu) (net 57))
-  (segment (start 148.844 125.08) (end 148.844 124.7648) (width 0.25) (layer F.Cu) (net 58))
-  (segment (start 148.844 124.7648) (end 149.86 123.7488) (width 0.25) (layer F.Cu) (net 58))
-  (segment (start 149.86 123.7488) (end 152.654 123.7488) (width 0.25) (layer F.Cu) (net 58))
-  (segment (start 152.654 123.7488) (end 153.67 122.7328) (width 0.25) (layer F.Cu) (net 58))
-  (segment (start 153.67 122.7328) (end 153.67 120.396) (width 0.25) (layer F.Cu) (net 58))
-  (segment (start 155.3972 118.6688) (end 156.9212 118.6688) (width 0.25) (layer F.Cu) (net 58))
-  (segment (start 153.67 120.396) (end 155.3972 118.6688) (width 0.25) (layer F.Cu) (net 58))
+  (segment (start 151.384 125.08) (end 166.004 125.08) (width 0.25) (layer F.Cu) (net 57))
+  (segment (start 168.0972 122.9868) (end 168.0972 121.158) (width 0.25) (layer F.Cu) (net 57))
+  (segment (start 166.004 125.08) (end 168.0972 122.9868) (width 0.25) (layer F.Cu) (net 57))
+  (segment (start 148.844 125.08) (end 150.099 123.825) (width 0.25) (layer F.Cu) (net 58))
+  (segment (start 150.099 123.825) (end 152.4508 123.825) (width 0.25) (layer F.Cu) (net 58))
+  (segment (start 152.4508 123.825) (end 153.2128 124.587) (width 0.25) (layer F.Cu) (net 58))
+  (segment (start 153.2128 124.587) (end 165.2016 124.587) (width 0.25) (layer F.Cu) (net 58))
+  (segment (start 165.2016 124.587) (end 166.5478 123.2408) (width 0.25) (layer F.Cu) (net 58))
+  (segment (start 166.5478 120.1674) (end 168.0972 118.618) (width 0.25) (layer F.Cu) (net 58))
+  (segment (start 166.5478 123.2408) (end 166.5478 120.1674) (width 0.25) (layer F.Cu) (net 58))
   (segment (start 140.0556 61.8852) (end 141.6704 61.8852) (width 0.25) (layer F.Cu) (net 64))
   (segment (start 141.6704 61.8852) (end 142.9258 60.6298) (width 0.25) (layer F.Cu) (net 64))
