File: pcb_files/mouse/mouse_v2.kicad_pcb (KiCad board)
At the start: 2 copper layers, 84.9 x 94.9 mm, 66 parts, among them J1 Conn_01x06_Female, J2 Conn_01x02_Female, J4 I2C_Conn, M1 Motor_DC, M2 Motor_DC, Q0 Q_Photo_NPN, Q1 Q_Photo_NPN, Q2 Q_Photo_NPN, Q3 Q_Photo_NPN, T0 Q_NMOS_DGS, T1 Q_NMOS_DGS, T2 Q_NMOS_DGS, T3 Q_NMOS_DGS, T4 Q_NMOS_DGS, U1 Teensy4.0, U2 SN754410NE (Half-Bridge), U3 LM1085-5.0, U4 Encoder_3081, U5 Encoder_3081

Commit message: traces update
Parts:
- moved SK4 112.0 mm to (160.1, 136.1)
- moved SK3 90.6 mm to (160.1, 58.0)
- moved SK1 2.90 mm to (160.1, 61.9)
Routing:
- net /5v: track 496.6 -> 454.6 mm, vias 2 -> 1
- net /3.3v: track 74.0 -> 104.6 mm
- net /LED_2: track 91.9 -> 91.4 mm
- net /LED_1: track 86.4 -> 85.8 mm
- net /GND: vias 48 -> 46

Commit message: updates
Parts:
- moved MH2 7.50 mm to (139.3, 113.4)
- moved MH1 7.24 mm to (181.2, 113.4)
- moved J4 2.02 mm to (181.2, 72.5)
Routing:
- net /vBatt: track 54.1 -> 51.2 mm
- net /Emitter_0: track 33.7 -> 36.2 mm
- net /VUSB: track 74.9 -> 76.9 mm
- net /GND: vias 46 -> 49

Commit message: added hc05 key jumper
Parts:
- added J3: Conn_01x02_Male, Connector_PinHeader_2.54mm:PinHeader_1x02_P2.54mm_Vertical, F.Cu at (136.1, 136.9)
Routing:
- net /HC05_KEY: track 0.00 -> 42.6 mm, vias 0 -> 1
- net /5v: track 454.6 -> 456.9 mm
- net Net-(R11-Pad1): track 11.8 -> 10.3 mm
- net Net-(D2-Pad1): track 17.3 -> 18.6 mm
- net /Emitter_2: track 49.8 -> 49.2 mm
- net /GND: vias 49 -> 47

Commit message: updated labels
Other:
- board text added: "USB"

Commit message: updates
Other:
- board text added: "J. Low, C. Diaz Kit-Mouse v1 2020"
- board text removed: "J. Low, C. Diaz Kit-Mouse v0 2020"

Commit message: changed led to smaller footprint, generated gerbers
Parts:
- D4, D5, D6: footprint LED_SMD:LED_1206_3216Metric_Pad1.42x1.75mm_HandSolder -> LED_SMD:LED_0201_0603Metric_Pad0.64x0.40mm_HandSolder
Routing:
- net /GND: track 28.5 -> 44.5 mm
- net Net-(D6-Pad2): track 2.93 -> 4.01 mm
- net Net-(D5-Pad2): track 2.93 -> 4.01 mm
- net Net-(D4-Pad2): track 2.93 -> 4.01 mm
